File: pcb/USBLabTool/Oscilloscope_FrontEnd.kicad_sch (KiCad schematic)
At the start: 88 parts, among them K1 G5V-2, K2 G5V-2, U1 AQY284SX, U2 AQY284SX, U3 CD74HC4316, U4 LMP7718, U5 CD74HC4316, U6 LMP7718, U7 OPA863, U8 OPA863

Commit message: push new layout
Connections:
- net +3.3VA: now also D3.2 (A), D4.2 (A); no longer D3.1 (K), D4.1 (K)
- net GNDA: now also D3.1 (K), D4.1 (K); no longer D3.2 (A), D4.2 (A)
Other:
- moved on the sheet: D3, D4
Changed lines of the file:
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@@
 	(symbol
 		(lib_id "Diode:BAV99")
-		(at 294.64 175.26 180)
+		(at 294.64 175.26 0)
+		(mirror x)
 		(unit 1)
 		(exclude_from_sim no)
@@
 		(on_board yes)
 		(dnp no)
-		(fields_autoplaced yes)
 		(property "Reference" "D3"
 			(at 294.64 179.07 0)
@@
 	(symbol
 		(lib_id "Diode:BAV99")
-		(at 304.8 63.5 180)
+		(at 304.8 63.5 0)
+		(mirror x)
 		(unit 1)
 		(exclude_from_sim no)
@@
 		(on_board yes)
 		(dnp no)
-		(fields_autoplaced yes)
 		(property "Reference" "D4"
 			(at 304.8 67.31 0)

Commit message: merge from V2
Parts:
- added TP15, TP18, TP19, TP20, TP21, TP22, TP23: TestPoint, TestPoint:TestPoint_Pad_2.0x2.0mm, symbol Connector:TestPoint
- TP7: footprint TestPoint:TestPoint_Pad_D2.0mm -> TestPoint:TestPoint_Pad_2.0x2.0mm
Connections:
- net CH0_ACDC: now also TP23.1
- net CH0_amp_1: now also TP18.1
- net CH0_amp_10: now also TP21.1
- net CH0_amp_2.5: now also TP19.1
- net CH0_amp_5: now also TP20.1
- net CH0_attenuate: now also TP22.1
- net TIM2_CH2: now also TP15.1
