File: pcb/USBLabTool/USB_USER.kicad_sch (KiCad schematic)
At the start: 17 parts, among them J20 USB_C_Receptacle, Q1 STL11N3LLH6, U17 TCPP01-M12, U19 USBLC6-2SC6

Commit message: 1
Parts:
- added JP3, JP4, JP5: SJ, Jumper:SolderJumper-2_P1.3mm_Open_RoundedPad1.0x1.5mm, symbol Jumper:SolderJumper_2_Open
Connections:
- net +5V: now also JP3.1 (A); no longer C70.1, C74.2, D10.2 (A), D9.C, J20.A4 (VBUS), J20.A9 (VBUS), J20.B4 (VBUS), J20.B9 (VBUS), Q1.5 (D), R67.1
- net UCPD_CC1: now also JP4.1 (A); no longer C72.2, J20.A5 (CC1), U17.7 (CC1c)
- net UCPD_CC2: now also JP5.1 (A); no longer C73.2, J20.B5 (CC2), U17.9 (CC2c)
- new net: C70.1, C74.2, D10.2 (A), D9.C, J20.A4 (VBUS), J20.A9 (VBUS), J20.B4 (VBUS), J20.B9 (VBUS), JP3.2 (B), Q1.5 (D), R67.1
- new net: C72.2, J20.A5 (CC1), JP4.2 (B), U17.7 (CC1c)
- new net: C73.2, J20.B5 (CC2), JP5.2 (B), U17.9 (CC2c)

Commit message: fixes
Parts:
- C70: value 10nF -> DNF
Other:
- note added: "10nF"
Changed lines of the file:
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@@
 	(generator_version "9.0")
 	(paper "A4")
+	(text "10nF"
+		(exclude_from_sim no)
+		(at 125.476 61.468 0)
+		(effects
+			(font
+				(size 1.27 1.27)
+			)
+		)
+	)
 	(junction
 		(at 234.95 134.62)
@@
 	)
 	(junction
+		(at 153.67 124.46)
+		(diameter 0)
+		(color 0 0 0 0)
+	)
+	(junction
 		(at 83.82 40.64)
 		(diameter 0)
@@
 	)
 	(junction
-		(at 88.9 57.15)
+		(at 168.91 124.46)
 		(diameter 0)
 		(color 0 0 0 0)
 	)
 	(junction
-		(at 175.26 39.37)
+		(at 171.45 121.92)
 		(diameter 0)
 		(color 0 0 0 0)
 	)
 	(junction
-		(at 217.17 64.77)
+		(at 88.9 57.15)
 		(diameter 0)
 		(color 0 0 0 0)
 	)
 	(junction
-		(at 218.44 53.34)
+		(at 175.26 39.37)
 		(diameter 0)
 		(color 0 0 0 0)
 	)
 	(junction
-		(at 233.68 57.15)
+		(at 217.17 64.77)
 		(diameter 0)
 		(color 0 0 0 0)
 	)
 	(junction
-		(at 142.24 72.39)
+		(at 218.44 53.34)
 		(diameter 0)
 		(color 0 0 0 0)
 	)
 	(junction
-		(at 151.13 121.92)
+		(at 233.68 57.15)
 		(diameter 0)
 		(color 0 0 0 0)
 	)
 	(junction
-		(at 153.67 124.46)
+		(at 142.24 72.39)
 		(diameter 0)
 		(color 0 0 0 0)
@@
 		(color 0 0 0 0)
 	)
+	(junction
+		(at 152.4 121.92)
+		(diameter 0)
+		(color 0 0 0 0)
+	)
 	(no_connect
 		(at 215.9 107.95)
@@
 	(wire
 		(pts
-			(xy 151.13 133.35) (xy 151.13 121.92)
+			(xy 152.4 133.35) (xy 152.4 121.92)
 		)
 		(stroke
@@
 	(wire
 		(pts
-			(xy 153.67 124.46) (xy 168.91 124.46)
-		)
-		(stroke
-			(width 0)
-			(type default)
-		)
-	)
-	(wire
-		(pts
 			(xy 238.76 52.07) (xy 238.76 57.15)
 		)
@@
 	(wire
 		(pts
-			(xy 151.13 121.92) (xy 171.45 121.92)
-		)
-		(stroke
-			(width 0)
-			(type default)
-		)
-	)
-	(wire
-		(pts
 			(xy 143.51 100.33) (xy 143.51 107.95)
 		)
@@
 	(wire
 		(pts
-			(xy 156.21 133.35) (xy 151.13 133.35)
+			(xy 156.21 133.35) (xy 152.4 133.35)
 		)
 		(stroke
@@
 	(wire
 		(pts
+			(xy 149.86 121.92) (xy 152.4 121.92)
+		)
+		(stroke
+			(width 0)
+			(type default)
+		)
+	)
+	(wire
+		(pts
 			(xy 142.24 72.39) (xy 142.24 85.09)
 		)
@@
 	(wire
 		(pts
-			(xy 148.59 121.92) (xy 151.13 121.92)
+			(xy 77.47 40.64) (xy 83.82 40.64)
 		)
 		(stroke
@@
 	(wire
 		(pts
-			(xy 77.47 40.64) (xy 83.82 40.64)
+			(xy 149.86 124.46) (xy 153.67 124.46)
 		)
 		(stroke
@@
 	(wire
 		(pts
+			(xy 168.91 124.46) (xy 153.67 124.46)
+		)
+		(stroke
+			(width 0)
+			(type default)
+		)
+	)
+	(wire
+		(pts
 			(xy 140.97 92.71) (xy 153.67 92.71)
 		)
@@
 	(wire
 		(pts
-			(xy 148.59 124.46) (xy 153.67 124.46)
+			(xy 172.72 124.46) (xy 168.91 124.46)
+		)
+		(stroke
+			(width 0)
+			(type default)
+		)
+	)
+	(wire
+		(pts
+			(xy 152.4 121.92) (xy 171.45 121.92)
 		)
 		(stroke
@@
 	(wire
 		(pts
+			(xy 171.45 121.92) (xy 172.72 121.92)
+		)
+		(stroke
+			(width 0)
+			(type default)
+		)
+	)
+	(wire
+		(pts
 			(xy 140.97 95.25) (xy 148.59 95.25)
 		)
@@
 	(global_label "USB_D-"
 		(shape input)
-		(at 148.59 124.46 180)
+		(at 172.72 124.46 0)
+		(fields_autoplaced yes)
+		(effects
+			(font
+				(size 1.27 1.27)
+			)
+			(justify left)
+		)
+		(property "Intersheetrefs" "${INTERSHEET_REFS}"
+			(at 183.3252 124.46 0)
+			(effects
+				(font
+					(size 1.27 1.27)
+				)
+				(justify left)
+				(hide yes)
+			)
+		)
+	)
+	(global_label "USB_FS_N"
+		(shape input)
+		(at 149.86 124.46 180)
 		(fields_autoplaced yes)
 		(effects
@@
 		)
 		(property "Intersheetrefs" "${INTERSHEET_REFS}"
-			(at 137.9848 124.46 0)
+			(at 137.501 124.46 0)
 			(effects
 				(font
@@
 		)
 	)
+	(global_label "USB_FS_P"
+		(shape input)
+		(at 149.86 121.92 180)
+		(fields_autoplaced yes)
+		(effects
+			(font
+				(size 1.27 1.27)
+			)
+			(justify right)
+		)
+		(property "Intersheetrefs" "${INTERSHEET_REFS}"
+			(at 137.5615 121.92 0)
+			(effects
+				(font
+					(size 1.27 1.27)
+				)
+				(justify right)
+				(hide yes)
+			)
+		)
+	)
 	(global_label "USCPD_DBn"
 		(shape input)
@@
 	(global_label "USB_D+"
 		(shape input)
-		(at 148.59 121.92 180)
+		(at 172.72 121.92 0)
 		(fields_autoplaced yes)
 		(effects
@@
 				(size 1.27 1.27)
 			)
-			(justify right)
+			(justify left)
 		)
 		(property "Intersheetrefs" "${INTERSHEET_REFS}"
-			(at 137.9848 121.92 0)
+			(at 183.3252 121.92 0)
 			(effects
 				(font
 					(size 1.27 1.27)
 				)
-				(justify right)
+				(justify left)
 				(hide yes)
 			)
@@
 			)
 		)
-		(property "Value" "10nF"
+		(property "Value" "DNF"
 			(at 118.11 61.468 90)
 			(effects

Commit message: PCB V2 updates
Changed lines of the file:
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@@
-	)
-	(junction
-		(at 153.67 124.46)
-		(diameter 0)
-		(color 0 0 0 0)
 	)
 	(junction
@@
 	(junction
 		(at 73.66 85.09)
-		(diameter 0)
-		(color 0 0 0 0)
-	)
-	(junction
-		(at 152.4 121.92)
 		(diameter 0)
 		(color 0 0 0 0)
@@
 	(wire
 		(pts
-			(xy 152.4 133.35) (xy 152.4 121.92)
+			(xy 151.13 133.35) (xy 151.13 121.92)
 		)
 		(stroke
@@
 	(wire
 		(pts
-			(xy 156.21 133.35) (xy 152.4 133.35)
+			(xy 151.13 121.92) (xy 171.45 121.92)
+		)
+		(stroke
+			(width 0)
+			(type default)
+		)
+	)
+	(wire
+		(pts
+			(xy 156.21 133.35) (xy 151.13 133.35)
 		)
 		(stroke
@@
 	(wire
 		(pts
-			(xy 149.86 121.92) (xy 152.4 121.92)
-		)
-		(stroke
-			(width 0)
-			(type default)
-		)
-	)
-	(wire
-		(pts
 			(xy 142.24 72.39) (xy 142.24 85.09)
 		)
@@
 	(wire
 		(pts
-			(xy 149.86 124.46) (xy 153.67 124.46)
-		)
-		(stroke
-			(width 0)
-			(type default)
-		)
-	)
-	(wire
-		(pts
 			(xy 116.84 107.95) (xy 143.51 107.95)
 		)
@@
 		(pts
 			(xy 172.72 124.46) (xy 168.91 124.46)
-		)
-		(stroke
-			(width 0)
-			(type default)
-		)
-	)
-	(wire
-		(pts
-			(xy 152.4 121.92) (xy 171.45 121.92)
 		)
 		(stroke
@@
 		)
 	)
-	(global_label "USB_FS_N"
-		(shape input)
-		(at 149.86 124.46 180)
-		(fields_autoplaced yes)
-		(effects
-			(font
-				(size 1.27 1.27)
-			)
-			(justify right)
-		)
-		(property "Intersheetrefs" "${INTERSHEET_REFS}"
-			(at 137.501 124.46 0)
-			(effects
-				(font
-					(size 1.27 1.27)
-				)
-				(justify right)
-				(hide yes)
-			)
-		)
-	)
 	(global_label "UCPD_CC1"
 		(shape input)
@@
 			(effects
 				(font
-					(size 1.27 1.27)
-				)
-				(justify right)
-				(hide yes)
-			)
-		)
-	)
-	(global_label "USB_FS_P"
-		(shape input)
-		(at 149.86 121.92 180)
-		(fields_autoplaced yes)
-		(effects
-			(font
-				(size 1.27 1.27)
-			)
-			(justify right)
-		)
-		(property "Intersheetrefs" "${INTERSHEET_REFS}"
-			(at 137.5615 121.92 0)
-			(effects
-				(font

Commit message: update pcb v2
Parts:
- added C69: 100n, Capacitor_SMD:C_0603_1608Metric_Pad1.08x0.95mm_HandSolder, symbol Device:C
Connections:
- net +5VCLEAN: now also C69.1
- net GNDA: now also C69.2
Changed lines of the file:
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@@
 	)
 	(junction
+		(at 125.73 142.24)
+		(diameter 0)
+		(color 0 0 0 0)
+	)
+	(junction
 		(at 148.59 95.25)
 		(diameter 0)
@@
 	(wire
 		(pts
+			(xy 125.73 142.24) (xy 132.08 142.24)
+		)
+		(stroke
+			(width 0)
+			(type default)
+		)
+	)
+	(wire
+		(pts
 			(xy 238.76 52.07) (xy 238.76 57.15)
 		)
@@
 	(wire
 		(pts
-			(xy 114.3 142.24) (xy 121.92 142.24)
+			(xy 114.3 142.24) (xy 125.73 142.24)
 		)
 		(stroke
@@
 	(global_label "+5VCLEAN"
 		(shape output)
-		(at 121.92 142.24 0)
+		(at 132.08 142.24 0)
 		(fields_autoplaced yes)
 		(effects
@@
 		)
 		(property "Intersheetrefs" "${INTERSHEET_REFS}"
-			(at 134.6419 142.24 0)
+			(at 144.8019 142.24 0)
 			(effects
 				(font
@@
 	)
 	(symbol
+		(lib_id "power:GNDA")
+		(at 125.73 149.86 0)
+		(unit 1)
+		(exclude_from_sim no)
+		(in_bom yes)
+		(on_board yes)
+		(dnp no)
+		(fields_autoplaced yes)
+		(property "Reference" "#PWR0127"
+			(at 125.73 156.21 0)
+			(effects
+				(font
+					(size 1.27 1.27)
+				)
+				(hide yes)
+			)
+		)
+		(property "Value" "GNDA"
+			(at 125.73 154.94 0)
+			(effects
+				(font
+					(size 1.27 1.27)
+				)
+			)
+		)
+		(property "Footprint" ""
+			(at 125.73 149.86 0)
+			(effects
+				(font
+					(size 1.27 1.27)
+				)
+				(hide yes)
+			)
+		)
+		(property "Datasheet" ""
+			(at 125.73 149.86 0)
+			(effects
+				(font
+					(size 1.27 1.27)
+				)
+				(hide yes)
+			)
+		)
+		(property "Description" "Power symbol creates a global label with name \"GNDA\" , analog ground"
+			(at 125.73 149.86 0)
+			(effects
+				(font
+					(size 1.27 1.27)
+				)
+				(hide yes)
+			)
+		)
+		(pin "1"
+		)
+		(instances
+			(project "USBLabTool"
+				(path "/b5440f7d-90d5-417e-adc2-aa6b11e5424d/37e12e55-0596-42de-ac66-6f566cb1a838"
+					(reference "#PWR0127")
+					(unit 1)
+				)
+			)
+		)
+	)
+	(symbol
 		(lib_id "USBLabTool:ESDA25P35-1U1M")
 		(at 234.95 101.6 90)
@@
 					(unit 1)
 				)
+			)
+		)
+	)
+	(symbol
+		(lib_id "Device:C")
+		(at 125.73 146.05 0)
+		(unit 1)
+		(exclude_from_sim no)
+		(in_bom yes)
+		(on_board yes)
+		(dnp no)
+		(property "Reference" "C69"
+			(at 129.032 145.034 0)
+			(effects
+				(font
+					(size 1.27 1.27)
+				)
+				(justify left)
+			)
+		)
+		(property "Value" "100n"
+			(at 127.762 148.336 0)
+			(effects
+				(font
+					(size 1.27 1.27)
+				)
+				(justify left)
+			)
+		)
+		(property "Footprint" "Capacitor_SMD:C_0603_1608Metric_Pad1.08x0.95mm_HandSolder"
+			(at 126.6952 149.86 0)
+			(effects
+				(font
+					(size 1.27 1.27)
+				)
+				(hide yes)
+			)
+		)
+		(property "Datasheet" "~"
+			(at 125.73 146.05 0)
+			(effects
+				(font
+					(size 1.27 1.27)
+				)
+				(hide yes)
+			)
+		)
+		(property "Description" ""
+			(at 125.73 146.05 0)
+			(effects
+				(font
+					(size 1.27 1.27)
+				)
+				(hide yes)
+			)
+		)
+		(pin "1"
+		)
+		(pin "2"
+		)
+		(instances
+			(project "USBLabTool"
+				(path "/b5440f7d-90d5-417e-adc2-aa6b11e5424d/37e12e55-0596-42de-ac66-6f566cb1a838"
+					(reference "C69")
+					(unit 1)
+				)
