File: pcb/USBLabTool/USB_USER.kicad_sch (KiCad schematic)
At the start: 17 parts, among them J20 USB_C_Receptacle, Q1 STL11N3LLH6, U17 TCPP01-M12, U19 USBLC6-2SC6

Commit message: push new layout
Parts:
- added JP3, JP4, JP5: SJ, Jumper:SolderJumper-2_P1.3mm_Open_RoundedPad1.0x1.5mm, symbol Jumper:SolderJumper_2_Open
Connections:
- net +5V: now also JP5.1 (A); no longer C70.1, C74.2, D10.2 (A), D9.C, J20.A4 (VBUS), J20.A9 (VBUS), J20.B4 (VBUS), J20.B9 (VBUS), Q1.5 (D), R67.1
- net UCPD_CC1: now also JP3.1 (A); no longer C72.2, J20.A5 (CC1), U17.7 (CC1c)
- net UCPD_CC2: now also JP4.1 (A); no longer C73.2, J20.B5 (CC2), U17.9 (CC2c)
- new net: C70.1, C74.2, D10.2 (A), D9.C, J20.A4 (VBUS), J20.A9 (VBUS), J20.B4 (VBUS), J20.B9 (VBUS), JP5.2 (B), Q1.5 (D), R67.1
- new net: C72.2, J20.A5 (CC1), JP3.2 (B), U17.7 (CC1c)
- new net: C73.2, J20.B5 (CC2), JP4.2 (B), U17.9 (CC2c)

Commit message: merge from V2
Parts:
- added C69: 100n, Capacitor_SMD:C_0603_1608Metric_Pad1.08x0.95mm_HandSolder, symbol Device:C
- C70: value 10nF -> DNF
Connections:
- net +5V: now also JP3.1 (A); no longer JP5.1 (A)
- net +5VCLEAN: now also C69.1
- net GNDA: now also C69.2
- net UCPD_CC1: now also JP4.1 (A); no longer JP3.1 (A)
- net UCPD_CC2: now also JP5.1 (A); no longer JP4.1 (A)
- net at C70.1, C74.2, D10.2 (A)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: now also JP3.2 (B); no longer JP5.2 (B)
- net at C72.2, J20.A5 (CC1), U17.7 (CC1c): now also JP4.2 (B); no longer JP3.2 (B)
- net at C73.2, J20.B5 (CC2), U17.9 (CC2c): now also JP5.2 (B); no longer JP4.2 (B)
Other:
- note added: "10nF"
