File: pcb/USBLabTool/Microcontroller.kicad_sch (KiCad schematic)
At the start: 27 parts, among them J1 Conn_01x06_Pin, J2 Conn_02x12_Odd_Even, SW1 TS02-66-73-BK-100-SCR-D, U12 STM32H563VITx, Y1 32.768kHz, Y2 NX2016SA-25M-EXS00A-CS08742

Commit message: update footprint
Parts:
- CR1: footprint SOD882_STM -> Diode_SMD:D_SOD-882
