File: pcb/USBLabTool/USBLabTool.kicad_pcb (KiCad board)
At the start: 4 copper layers, 237 parts, among them J1 Conn_01x06_Pin, J17 2x01, J19 T_N5V, J2 Conn_02x12_Odd_Even, J20 USB_C_Receptacle, K1 G5V-2, K2 G5V-2, Q1 STL11N3LLH6, SW1 TS02-66-73-BK-100-SCR-D, U1 AQY284SX, U10 MC33274ADR2G, U11 DG403, U12 STM32H563VITx, U13 R1283K002A, U14 ST1L05APU33R, U15 ST1L05APU33R, U16 LTC1983ES6-5TRMPBF, U17 TCPP01-M12, U18 74HC245, U19 USBLC6-2SC6, U2 AQY284SX, U20 74HC245, U3 CD74HC4316, U4 LMP7718, U5 CD74HC4316, U6 LMP7718, U7 OPA863, U8 OPA863, U9 MC33274ADR2G, Y1 32.768kHz, Y2 NX2016SA-25M-EXS00A-CS08742

Commit message: pcb update
Parts:
- turned U12 to 180 degrees
Routing:
- net ADC1_INP0: track 30.6 -> 14.3 mm
- net +3.3V: track 103.3 -> 87.8 mm, vias 9 -> 7
- net TIM2_CH2: track 15.8 -> 8.25 mm
- net VREFP: track 7.57 -> 0.00 mm
- net Net-(U12-VDDA): track 6.65 -> 1.53 mm
- net GND: track 322.4 -> 317.6 mm, vias 37 -> 35
- net Net-(C31-Pad1): track 17.9 -> 14.0 mm
- net RCC_OSC32_IN: track 22.3 -> 25.7 mm, vias 0 -> 1
- net unconnected-(U12-PE11-Pad42): track 0.00 -> 2.51 mm, vias 0 -> 1
- net TIM1_CH1: track 3.05 -> 0.53 mm, vias 1 -> 0
- net Net-(C31-Pad2): track 11.0 -> 8.55 mm
- net RCC_OSC32_OUT: track 19.2 -> 21.1 mm, vias 0 -> 1
- net LOGIC_IN4: track 0.00 -> 1.45 mm, vias 0 -> 1
- net UCPD_CC2: track 26.6 -> 26.0 mm
- net NRST: track 70.5 -> 71.0 mm

Commit message: update footprint
Parts:
- added C78: 100nF, Capacitor_SMD:C_0603_1608Metric, F.Cu at (181.6, 87.0)
- CR1: footprint userfp:SOD882_STM -> Diode_SMD:D_SOD-882
Connections:
- U12 pad 1: UCPD_CC2 -> unconnected-(U12-PE2-Pad1)
- U12 pad 2: UCPD_CC1 -> unconnected-(U12-PE3-Pad2)
- U12 pad 45: unconnected-(U12-PE14-Pad45) -> CH0_attenuate
- U12 pad 46: unconnected-(U12-PE15-Pad46) -> CH1_attenuate
- U12 pad 52: CH0_attenuate -> UCPD_CC1
- U12 pad 53: CH1_attenuate -> UCPD_CC2
