File: pcb/USBLabTool/Power_Supply.kicad_sch (KiCad schematic)
At the start: 54 parts, among them J19 T_N5V, U10 MC33274ADR2G, U11 DG403, U13 R1283K002A, U14 ST1L05APU33R, U15 ST1L05APU33R, U16 LTC1983ES6-5TRMPBF, U9 MC33274ADR2G

Commit message: push new layout
Changed lines of the file:
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@@
 	(text "Negative 5V Power supply"
 		(exclude_from_sim no)
-		(at 179.6288 19.9136 0)
+		(at 198.628 19.05 0)
 		(effects
 			(font

Commit message: merge from V2
Parts:
- C57: value 100n -> 10u
- C59, C60: value 4.7uF -> 100nF
- L5, L6: value 47uH -> 4.7uH; footprint Inductor_SMD:L_0603_1608Metric_Pad1.05x0.95mm_HandSolder -> userfp:IND_TAIYO_NRH2410_TAY
Changed lines of the file:
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@@
 	(text "Negative 5V Power supply"
 		(exclude_from_sim no)
-		(at 198.628 19.05 0)
+		(at 179.6288 19.9136 0)
 		(effects
 			(font
@@
 	(wire
 		(pts
-			(xy 137.16 39.37) (xy 137.16 44.45)
+			(xy 137.16 39.37) (xy 137.16 43.18)
 		)
 		(stroke
@@
 	(wire
 		(pts
-			(xy 250.19 67.31) (xy 252.73 67.31)
-		)
-		(stroke
-			(width 0)
-			(type default)
-		)
-	)
-	(wire
-		(pts
 			(xy 133.35 96.52) (xy 133.35 153.67)
 		)
@@
 	(wire
 		(pts
+			(xy 250.19 67.31) (xy 264.16 67.31)
+		)
+		(stroke
+			(width 0)
+			(type default)
+		)
+	)
+	(wire
+		(pts
 			(xy 59.69 82.55) (xy 62.23 82.55)
 		)
@@
 	(wire
 		(pts
-			(xy 64.77 133.35) (xy 46.99 133.35)
+			(xy 46.99 133.35) (xy 64.77 133.35)
 		)
 		(stroke
@@
 	(wire
 		(pts
-			(xy 124.46 39.37) (xy 124.46 44.45)
+			(xy 124.46 39.37) (xy 124.46 43.18)
 		)
 		(stroke
@@
 	(global_label "-5VCLEAN"
 		(shape output)
-		(at 252.73 67.31 0)
+		(at 264.16 67.31 0)
 		(fields_autoplaced yes)
 		(effects
@@
 		)
 		(property "Intersheetrefs" "${INTERSHEET_REFS}"
-			(at 265.4519 67.31 0)
+			(at 276.8819 67.31 0)
 			(effects
 				(font
@@
 			)
 		)
-		(property "Value" "47uH"
+		(property "Value" "4.7uH"
 			(at 166.624 128.016 90)
 			(effects
@@
 			)
 		)
-		(property "Footprint" "Inductor_SMD:L_0603_1608Metric_Pad1.05x0.95mm_HandSolder"
+		(property "Footprint" "userfp:IND_TAIYO_NRH2410_TAY"
 			(at 166.37 130.81 0)
 			(effects
@@
 			)
 		)
+		(property "Purpose" ""
+			(at 166.37 130.81 0)
+			(effects
+				(font
+					(size 1.27 1.27)
+				)
+				(hide yes)
+			)
+		)
 		(pin "1"
 		)
@@
 			)
 		)
-		(property "Value" "4.7uF"
+		(property "Value" "100nF"
 			(at 180.848 119.126 0)
 			(effects
@@
 	(symbol
 		(lib_id "power:GNDA")
-		(at 137.16 44.45 0)
+		(at 137.16 43.18 0)
 		(unit 1)
 		(exclude_from_sim no)
@@
 		(fields_autoplaced yes)
 		(property "Reference" "#PWR0111"
-			(at 137.16 50.8 0)
+			(at 137.16 49.53 0)
 			(effects
 				(font
@@
 		)
 		(property "Value" "GNDA"
-			(at 137.16 49.53 0)
+			(at 137.16 48.26 0)
 			(effects
 				(font
@@
 		)
 		(property "Footprint" ""
-			(at 137.16 44.45 0)
+			(at 137.16 43.18 0)
 			(effects
 				(font
@@
 		)
 		(property "Datasheet" ""
-			(at 137.16 44.45 0)
+			(at 137.16 43.18 0)
 			(effects
 				(font
@@
 		)
 		(property "Description" ""
-			(at 137.16 44.45 0)
+			(at 137.16 43.18 0)
 			(effects
 				(font
@@
 			)
 		)
-		(property "Value" "4.7uF"
+		(property "Value" "100nF"
 			(at 157.226 118.618 0)
 			(effects
@@
 	(symbol
 		(lib_id "power:GNDA")
-		(at 124.46 44.45 0)
+		(at 124.46 43.18 0)
 		(unit 1)
 		(exclude_from_sim no)
@@
 		(fields_autoplaced yes)
 		(property "Reference" "#PWR0108"
-			(at 124.46 50.8 0)
+			(at 124.46 49.53 0)
 			(effects
 				(font
@@
 		)
 		(property "Value" "GNDA"
-			(at 124.46 49.53 0)
+			(at 124.46 48.26 0)
 			(effects
 				(font
@@
 		)
 		(property "Footprint" ""
-			(at 124.46 44.45 0)
+			(at 124.46 43.18 0)
 			(effects
 				(font
@@
 		)
 		(property "Datasheet" ""
-			(at 124.46 44.45 0)
+			(at 124.46 43.18 0)
 			(effects
 				(font
@@
 		)
 		(property "Description" ""
-			(at 124.46 44.45 0)
+			(at 124.46 43.18 0)
 			(effects
 				(font
@@
 			)
 		)
-		(property "Value" "47uH"
+		(property "Value" "4.7uH"
 			(at 166.116 110.744 90)
 			(effects
@@
 			)
 		)
-		(property "Footprint" "Inductor_SMD:L_0603_1608Metric_Pad1.05x0.95mm_HandSolder"
+		(property "Footprint" "userfp:IND_TAIYO_NRH2410_TAY"
 			(at 166.37 113.03 0)
 			(effects
@@
 			)
 		)
+		(property "Purpose" ""
+			(at 166.37 113.03 0)
+			(effects
+				(font
+					(size 1.27 1.27)
+				)
+				(hide yes)
+			)
+		)
 		(pin "1"
 		)
@@
 			)
 		)
-		(property "Value" "100n"
+		(property "Value" "10u"
 			(at 140.97 36.8299 0)
 			(effects
